File: project-tmp117.kicad_pcb (KiCad board)
At the start: 2 copper layers, 40.5 x 14 mm, 16 parts, among them J1 Conn_01x01_Pin, J2 Conn_01x01_Pin, J3 Conn_01x01_Pin, J4 Conn_01x01_Pin, J5 Conn_01x01_Pin, J7 SM04B-SRSS-TB(LF)(SN), J8 SM04B-SRSS-TB(LF)(SN), U1 TMP117AIDRVR

Commit message: Add version
Other:
- board text added: "François Gervais 2 avril 2024 v1.0.0"
- board text removed: "François Gervais 2 avril 2024"
